File: PCBs/Buzzer/Buzzer.kicad_pcb (KiCad board)
At the start: 2 copper layers, 40 x 20 mm, 3 parts, among them J1 RJ45, J2 Conn_01x04_Pin, U1 ATtiny85-20P

Commit message: update footprint
Parts:
- J1: footprint Buzzer:WR-MJ Modular Jack Horizontal Shielded w. EMI Panel Finger 8P8C Tab Up -> Library:WR-MJ Modular Jack Horizontal Shielded w. EMI Panel Finger 8P8C Tab Up
Changed lines of the file:
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@@
 		)
 	)
-	(footprint "Buzzer:WR-MJ Modular Jack Horizontal Shielded w. EMI Panel Finger 8P8C Tab Up"
+	(footprint "Library:WR-MJ Modular Jack Horizontal Shielded w. EMI Panel Finger 8P8C Tab Up"
 		(layer "F.Cu")
 		(at 81.585 75.15 90)
 		(descr "WR-MJ Modular Jack Horizontal Shielded w. EMI Panel Finger 8P8C Tab Up")
 		(property "Reference" "J1"
-			(at -8.2675 -9.0425 90)
+			(at 10.1925 -6.485 90)
 			(unlocked yes)
 			(layer "F.SilkS")
@@
 		)
 		(property "Value" "RJ45"
-			(at -8.35 -6.585 90)
+			(at 10.11 -4.0275 90)
 			(unlocked yes)
 			(layer "F.Fab")
@@
 			)
 		)
-		(property "Footprint" "Buzzer:WR-MJ Modular Jack Horizontal Shielded w. EMI Panel Finger 8P8C Tab Up"
+		(property "Footprint" "Library:WR-MJ Modular Jack Horizontal Shielded w. EMI Panel Finger 8P8C Tab Up"
 			(at 0 0 90)
 			(layer "F.Fab")
