File: PCBs/Buzzer/Buzzer.kicad_sch (KiCad schematic)
At the start: 3 parts, among them J1 RJ45, J2 Conn_01x04_Pin, U1 ATtiny85-20P

Commit message: update footprint
Parts:
- J1: footprint Buzzer:WR-MJ Modular Jack Horizontal Shielded w. EMI Panel Finger 8P8C Tab Up -> Library:WR-MJ Modular Jack Horizontal Shielded w. EMI Panel Finger 8P8C Tab Up
Changed lines of the file:
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@@
 			)
 		)
-		(property "Footprint" "Buzzer:WR-MJ Modular Jack Horizontal Shielded w. EMI Panel Finger 8P8C Tab Up"
+		(property "Footprint" "Library:WR-MJ Modular Jack Horizontal Shielded w. EMI Panel Finger 8P8C Tab Up"
 			(at 121.92 64.135 90)
 			(effects
