File: PCBs/Sensor/Sensor.kicad_sch (KiCad schematic)
At the start: 7 parts, among them J1 RJ45, J2 RJ45, U1 ATtiny85-20P

Commit message: assigned footprints
Parts:
- D1: value LED -> green; footprint (none) -> LED_THT:LED_D5.0mm
- J1, J2: footprint (none) -> Sensor:WR-MJ Modular Jack Horizontal Shielded w. EMI Panel Finger 8P8C Tab Up
- R2: value R -> 220; footprint (none) -> Resistor_THT:R_Axial_DIN0204_L3.6mm_D1.6mm_P7.62mm_Horizontal
- R3: value R -> 10k; footprint (none) -> Resistor_THT:R_Axial_DIN0204_L3.6mm_D1.6mm_P7.62mm_Horizontal
Changed lines of the file:
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@@
 			)
 		)
-		(property "Footprint" ""
+		(property "Footprint" "Sensor:WR-MJ Modular Jack Horizontal Shielded w. EMI Panel Finger 8P8C Tab Up"
 			(at 142.24 56.515 90)
 			(effects
@@
 			)
 		)
-		(property "Value" "R"
+		(property "Value" "220"
 			(at 105.41 93.9799 0)
 			(effects
@@
 			)
 		)
-		(property "Footprint" ""
+		(property "Footprint" "Resistor_THT:R_Axial_DIN0204_L3.6mm_D1.6mm_P7.62mm_Horizontal"
 			(at 104.648 92.71 90)
 			(effects
@@
 			)
 		)
-		(property "Value" "LED"
+		(property "Value" "green"
 			(at 106.68 87.9474 90)
 			(effects
@@
 			)
 		)
-		(property "Footprint" ""
+		(property "Footprint" "LED_THT:LED_D5.0mm"
 			(at 102.87 85.09 0)
 			(effects
@@
 			)
 		)
-		(property "Value" "R"
+		(property "Value" "10k"
 			(at 78.74 85.09 90)
 			(effects
@@
 			)
 		)
-		(property "Footprint" ""
+		(property "Footprint" "Resistor_THT:R_Axial_DIN0204_L3.6mm_D1.6mm_P7.62mm_Horizontal"
 			(at 78.74 88.9 0)
 			(effects
@@
 			)
 		)
-		(property "Footprint" ""
+		(property "Footprint" "Sensor:WR-MJ Modular Jack Horizontal Shielded w. EMI Panel Finger 8P8C Tab Up"
 			(at 142.24 83.185 90)
 			(effects

Commit message: routing
Parts:
- R2: footprint Resistor_THT:R_Axial_DIN0204_L3.6mm_D1.6mm_P7.62mm_Horizontal -> Resistor_THT:R_Axial_DIN0207_L6.3mm_D2.5mm_P10.16mm_Horizontal
- R3: footprint Resistor_THT:R_Axial_DIN0204_L3.6mm_D1.6mm_P7.62mm_Horizontal -> Resistor_THT:R_Axial_DIN0207_L6.3mm_D2.5mm_P10.16mm_Horizontal; symbol pspice:R -> Device:R
Connections:
- no-connect marks 1 -> 0
Other:
- moved on the sheet: R3
Changed lines of the file:
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@@
 		(color 0 0 0 0)
-	)
-	(no_connect
-		(at 72.39 31.75)
 	)
 	(wire
@@
 			)
 		)
-		(property "Footprint" "Resistor_THT:R_Axial_DIN0204_L3.6mm_D1.6mm_P7.62mm_Horizontal"
+		(property "Footprint" "Resistor_THT:R_Axial_DIN0207_L6.3mm_D2.5mm_P10.16mm_Horizontal"
 			(at 104.648 92.71 90)
 			(effects
@@
 	(symbol
 		(lib_id "power:+5V")
-		(at 72.39 88.9 0)
+		(at 77.47 88.9 0)
 		(unit 1)
 		(exclude_from_sim no)
@@
 		(fields_autoplaced yes)
 		(property "Reference" "#PWR05"
-			(at 72.39 92.71 0)
+			(at 77.47 92.71 0)
 			(effects
 				(font
@@
 		)
 		(property "Value" "+5V"
-			(at 72.39 83.82 0)
+			(at 77.47 83.82 0)
 			(effects
 				(font
@@
 		)
 		(property "Footprint" ""
-			(at 72.39 88.9 0)
+			(at 77.47 88.9 0)
 			(effects
 				(font
@@
 		)
 		(property "Datasheet" ""
-			(at 72.39 88.9 0)
+			(at 77.47 88.9 0)
 			(effects
 				(font
@@
 		)
 		(property "Description" "Power symbol creates a global label with name \"+5V\""
-			(at 72.39 88.9 0)
+			(at 77.47 88.9 0)
 			(effects
 				(font
@@
 	)
 	(symbol
-		(lib_id "pspice:R")
-		(at 78.74 88.9 90)
+		(lib_id "Device:R")
+		(at 81.28 88.9 90)
 		(unit 1)
 		(exclude_from_sim no)
@@
 		(fields_autoplaced yes)
 		(property "Reference" "R3"
-			(at 78.74 82.55 90)
+			(at 81.28 82.55 90)
 			(effects
 				(font
@@
 		)
 		(property "Value" "10k"
-			(at 78.74 85.09 90)
-			(effects
-				(font
-					(size 1.27 1.27)
-				)
-			)
-		)
-		(property "Footprint" "Resistor_THT:R_Axial_DIN0204_L3.6mm_D1.6mm_P7.62mm_Horizontal"
-			(at 78.74 88.9 0)
+			(at 81.28 85.09 90)
+			(effects
+				(font
+					(size 1.27 1.27)
+				)
+			)
+		)
+		(property "Footprint" "Resistor_THT:R_Axial_DIN0207_L6.3mm_D2.5mm_P10.16mm_Horizontal"
+			(at 81.28 90.678 90)
 			(effects
 				(font
@@
 		)
 		(property "Datasheet" "~"
-			(at 78.74 88.9 0)
-			(effects
-				(font
-					(size 1.27 1.27)
-				)
-				(hide yes)
-			)
-		)
-		(property "Description" "Resistor symbol for simulation only"
-			(at 78.74 88.9 0)
-			(effects
-				(font
+			(at 81.28 88.9 0)
+			(effects
+				(font
+					(size 1.27 1.27)
+				)
+				(hide yes)
+			)
+		)
+		(property "Description" "Resistor"
+			(at 81.28 88.9 0)
+			(effects
+				(font

Commit message: added info text
Other:
- company: (none) -> Manuel König HHN HTWG x42.space
- title: (none) -> Laser-Parkour Sensor
Changed lines of the file:
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@@
 	(generator_version "8.0")
 	(paper "A4")
+	(title_block
+		(title "Laser-Parkour Sensor")
+		(date "2024-08-18")
+		(rev "01")
+		(company "Manuel König HHN HTWG x42.space")
+	)
 	(junction
 		(at 118.11 63.5)

Commit message: update footprint
Parts:
- J1, J2: footprint Sensor:WR-MJ Modular Jack Horizontal Shielded w. EMI Panel Finger 8P8C Tab Up -> Library:WR-MJ Modular Jack Horizontal Shielded w. EMI Panel Finger 8P8C Tab Up
Changed lines of the file:
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@@
 			)
 		)
-		(property "Footprint" "Sensor:WR-MJ Modular Jack Horizontal Shielded w. EMI Panel Finger 8P8C Tab Up"
+		(property "Footprint" "Library:WR-MJ Modular Jack Horizontal Shielded w. EMI Panel Finger 8P8C Tab Up"
 			(at 142.24 56.515 90)
 			(effects
@@
 			)
 		)
-		(property "Footprint" "Sensor:WR-MJ Modular Jack Horizontal Shielded w. EMI Panel Finger 8P8C Tab Up"
+		(property "Footprint" "Library:WR-MJ Modular Jack Horizontal Shielded w. EMI Panel Finger 8P8C Tab Up"
 			(at 142.24 83.185 90)
 			(effects
