File: PCBs/Controller/Controller.kicad_pcb (KiCad board)
At the start: 2 copper layers, 60 x 80 mm, 18 parts, among them J1 RJ45, J2 RJ45, J3 RJ45, J4 RJ45, J5 Barrel_Jack_Switch, J6 Conn_01x04_Pin, J7 Conn_01x03_Pin, SW1 RotaryEncoder_Switch, SW2 SW_Push, U1 Pico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

Commit message: better rj45 routing
Routing:
- net Net-(JP1-B): track 90.3 -> 79.1 mm, vias 3 -> 2
- net /SCL0: track 95.6 -> 100.9 mm, vias 3 -> 1
- net +3.3V: track 113.1 -> 110.2 mm, vias 3 -> 4
- net Net-(JP3-B): track 114.1 -> 114.7 mm
