File: PCBs/Controller/Controller.kicad_pcb (KiCad board)
At the start: 2 copper layers, 60 x 80 mm, 18 parts, among them J1 RJ45, J2 RJ45, J3 RJ45, J4 RJ45, J5 Barrel_Jack_Switch, J6 Conn_01x04_Pin, J7 Conn_01x03_Pin, SW1 RotaryEncoder_Switch, SW2 SW_Push, U1 Pico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

Commit message: Controller Rev. 01
Parts:
- removed C2: 22μ, Capacitor_THT:CP_Radial_D5.0mm_P2.00mm
- removed J7: Conn_01x03_Pin, Connector_PinHeader_2.54mm:PinHeader_1x03_P2.54mm_Vertical
- removed JP3: Jumper_2_Bridged, Jumper:SolderJumper-2_P1.3mm_Bridged_RoundedPad1.0x1.5mm
- removed U2: AMS1117-3.3, Package_TO_SOT_SMD:SOT-223-3_TabPin2
- added D1: LED_RKGB, LED_THT:LED_D5.0mm-4_RGB_Wide_Pins, F.Cu at (108.3, 103.0)
- added R1: 220, Resistor_THT:R_Axial_DIN0207_L6.3mm_D2.5mm_P10.16mm_Horizontal, F.Cu at (108.0, 98.5)
- added R2: 220, Resistor_THT:R_Axial_DIN0207_L6.3mm_D2.5mm_P10.16mm_Horizontal, F.Cu at (111.0, 98.5)
- added R3: 110, Resistor_THT:R_Axial_DIN0207_L6.3mm_D2.5mm_P10.16mm_Horizontal, F.Cu at (114.0, 98.5)
- added R4: 10k, Resistor_THT:R_Axial_DIN0207_L6.3mm_D2.5mm_P10.16mm_Horizontal, F.Cu at (114.3, 127.5)
- added R5: 10k, Resistor_THT:R_Axial_DIN0207_L6.3mm_D2.5mm_P10.16mm_Horizontal, F.Cu at (122.5, 110.5)
- added R6: 5k, Resistor_THT:R_Axial_DIN0207_L6.3mm_D2.5mm_P10.16mm_Horizontal, F.Cu at (143.0, 113.0)
- added U3: Level Converter, Library:Level_Converter, F.Cu at (141.0, 128.2)
- JP2: value Jumper_3_Bridged12 -> Jumper_2_Open; footprint Jumper:SolderJumper-3_P1.3mm_Bridged12_RoundedPad1.0x1.5mm -> Jumper:SolderJumper-2_P1.3mm_Open_RoundedPad1.0x1.5mm
- moved JP2 69.7 mm to (146.2, 123.0)
- moved BZ1 51.1 mm to (109.5, 75.0)
- moved SW2 29.3 mm to (133.5, 113.5)
- moved JP1 19.1 mm to (144.7, 128.0)
- moved J6 9.12 mm to (104.0, 100.2)
- moved C1 7.83 mm to (112.0, 67.0), turned to -90 degrees
- moved C3 3.00 mm to (143.5, 60.0)
Connections:
- J1 pad 3: Net-(JP3-B) -> Net-(JP1-B)
- J1 pad 4: +3.3V -> +5V
- J1 pad 5: +3.3V -> +5V
- J1 pad 6: Net-(JP1-B) -> Net-(JP2-B)
- J2 pad 3: Net-(JP3-B) -> Net-(JP1-B)
- J2 pad 4: +3.3V -> +5V
- J2 pad 5: +3.3V -> +5V
- J2 pad 6: Net-(JP1-B) -> Net-(JP2-B)
- J3 pad 3: Net-(JP3-B) -> Net-(JP1-B)
- J3 pad 4: +3.3V -> +5V
- J3 pad 5: +3.3V -> +5V
- J3 pad 6: Net-(JP1-B) -> Net-(JP2-B)
- J4 pad 3: Net-(JP3-B) -> Net-(JP1-B)
- J4 pad 4: +3.3V -> +5V
- J4 pad 5: +3.3V -> +5V
- J4 pad 6: Net-(JP1-B) -> Net-(JP2-B)
- JP1 pad 1: /FU -> /AT_RS
- JP2 pad 1: Net-(JP2-A) -> /FU
- JP2 pad 2: +3.3V -> Net-(JP2-B)
- U1 pad 10: unconnected-(U1-GPIO7-Pad10)_1 -> /RED
- U1 pad 11: unconnected-(U1-GPIO8-Pad11) -> /GREEN
- U1 pad 12: unconnected-(U1-GPIO9-Pad12)_1 -> /BLUE
- U1 pad 21: /SDA0 -> Net-(U1-GPIO16)
- U1 pad 22: /SCL0 -> Net-(U1-GPIO17)
- U1 pad 24: /AT_RS -> Net-(U1-GPIO18)
- U1 pad 25: /FU -> Net-(U1-GPIO19)
- U1 pad 27: /BZ1 -> unconnected-(U1-GPIO21-Pad27)_1
- U1 pad 41: Net-(J7-Pin_1) -> unconnected-(U1-SWCLK-Pad41)
- U1 pad 43: Net-(J7-Pin_3) -> unconnected-(U1-SWDIO-Pad43)_1
- U1 pad 7: unconnected-(U1-GPIO5-Pad7)_1 -> /BZ1
Routing:
- net Net-(JP3-B): track 114.7 -> 0.00 mm, vias 3 -> 0
- net +3.3V: track 110.1 -> 0.00 mm, vias 4 -> 0
- net +5V: track 114.6 -> 220.9 mm, vias 0 -> 4
- net Net-(JP2-B): track 0.00 -> 75.7 mm
- net Net-(JP2-A): track 58.1 -> 0.00 mm, vias 1 -> 0
- net /RUN: track 89.7 -> 37.4 mm
- net +3V3: track 13.4 -> 65.6 mm
- net Net-(U1-GPIO19): track 0.00 -> 27.2 mm
- net Net-(U1-GPIO18): track 0.00 -> 24.4 mm
- net Net-(JP1-B): track 79.1 -> 102.2 mm, vias 2 -> 3
- net Net-(U1-GPIO17): track 0.00 -> 21.1 mm
- net Net-(U1-GPIO16): track 0.00 -> 20.4 mm, vias 0 -> 1
- net /SDA0: track 86.2 -> 105.3 mm, vias 4 -> 3
- net /BZ1: track 31.1 -> 13.2 mm
- net /RED: track 0.00 -> 17.0 mm
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
Commit message: update pcb
Other:
- board text added: "Laser-Parkour Controller Rev. 02 © 2024 Manuel König HHN HTWG x42.space"
- board text removed: "Laser-Parkour Controller Rev. 01 © 2024 Manuel König HHN HTWG x42.space"

Commit message: Controller Rev. 02
Parts:
- removed C3: 0.1μ, Capacitor_THT:C_Disc_D3.0mm_W1.6mm_P2.50mm
- added D2: 1N4007, Diode_THT:D_DO-41_SOD81_P7.62mm_Horizontal, F.Cu at (115.0, 63.7)
- moved R4 10.2 mm to (124.5, 127.5), turned to 180 degrees
- moved R5 10.2 mm to (112.3, 110.5), turned to 0 degrees
- moved C1 3.37 mm to (109.0, 68.5)
Connections:
- R4 pad 1: GND -> +3V3
- R5 pad 1: /RE_B -> +3V3
- R5 pad 2: GND -> /RE_B
- U1 pad 39: +5V -> Net-(D2-K)
Routing:
- net +3V3: track 65.6 -> 109.4 mm
- net Net-(D2-K): track 0.00 -> 37.7 mm
- net +5V: track 220.9 -> 222.4 mm, vias 4 -> 5
